File: COMET-X.kicad_pcb (KiCad board)
At the start: 2 copper layers, 110 x 45 mm, 19 parts, among them J1 ATX_12V_IN, J2 10146065-113Y1LF, J3 G97R24312HR_EP, U2 TPS5450ddar

Commit message: update xschematic
Other:
- copper layers 2 -> 6
